File: Design/MainBoard_V1.1.sch (EAGLE design)
At the start: 61 parts, among them IC3 LM2936MP-3.3, Q1 8meg, Q2 2N3904, Q4 2N3704, X1 SDBMF

Commit message: Schematic Update
Parts:
- removed Q2: 2N3904, transistor-small-signal:2N3904
- removed U$1: STM32F20XR, stm32F:STM32F20XR
- removed U$2: MICRO-USB-SHIELD-ZX62R-B-5P, con-hirose:MICRO-USB-SHIELD-ZX62R-B-5P
- removed X1: SDBMF, farnell:SDBMF
- added MICRO_USB: MICRO-USB-SHIELD-ZX62R-B-5P, con-hirose:MICRO-USB-SHIELD-ZX62R-B-5P
- added R19, R20: 0, rcl:R-US_R0805
- added SD_CARD: SDBMF, farnell:SDBMF
- added SENSOR_ADC: (no value), con-lstb:MA03-1
- added SENSOR_I2C: (no value), con-lstb:MA04-1
- added TP9: TPB1,27, testpad:TPB1,27
- added U1: STM32F20XR, stm32F:STM32F20XR
- Q1: value 8meg -> 25meg
- R5: value 10k -> 22
Connections:
- removed net N$10 (its old number): Q2.B, R6.1, TP4.TP, U$1.JTMS/SWDIO/PA13
- removed net N$11 (its old number): D3.C, R7.1, TP5.TP, U$1.JTCK/SWCLK/PA14
- removed net N$12 (its old number): D5.C, Q2.E, R10.1, TP6.TP, U$1.JTDO/TRACESSW0/PB3
- removed net N$20: R9.1, U$1.PB2
- removed net N$22: R1.2, U$1.PH1/OSC_OUT
- removed net N$23: R11.2, U$1.PC9, X1.8
- removed net N$24: R12.2, U$1.PC8, X1.7
- removed net N$25: R13.2, U$1.PC11, X1.2
- removed net N$26: U$1.PA11, U$2G$2.2
- removed net N$27: U$1.PC12, X1.5
- removed net N$28: R15.2, U$1.PD2, X1.3
- removed net N$29: R18.1, U$1.PA12, U$2G$2.3
- removed net N$3: C5.1, Q1.2, U$1.PH0/OSC_IN
- removed net N$31: R14.2, U$1.PC10, X1.1
- removed net N$7: R2.2, TP8.TP, U$1.BOOT0
- removed net N$8 (its old number): D6.C, JTAG.3, Q2.C, TP2.TP, U$1.NJTRST/PB4
- removed net N$9: R8.1, TP3.TP, U$1.JTDI/PA15
- removed net VDD1: C14.2, C6.1, D4.C, JTAG.15, S1.3, S1.4, TP7.TP, U$1.NRST
- new net ADC1_IN1: SENSOR_ADC.2, U1.PA1
- new net BOOT0: R2.2, TP8.TP, U1.BOOT0
- new net BOOT1: R9.1, TP9.TP, U1.PB2
- new net DM: MICRO_USBG$2.2, U1.PA11
- new net DP: MICRO_USBG$2.3, R18.1, U1.PA12
- new net I2C1_SCL: R20.1, U1.PB6
- new net I2C1_SDA: R19.1, U1.PB7
- new net JTCK: D3.C, R7.1, TP5.TP, U1.JTCK/SWCLK/PA14
- new net JTDI: R8.1, TP3.TP, U1.JTDI/PA15
- new net JTDO: D5.C, R5.1, TP6.TP, U1.JTDO/TRACESSW0/PB3
- new net JTMS: R6.1, TP4.TP, U1.JTMS/SWDIO/PA13
- new net NJTRST: D6.C, JTAG.3, TP2.TP, U1.NJTRST/PB4
- new net OSC_IN: C5.1, Q1.2, U1.PH0/OSC_IN
- new net OSC_OUT: R1.2, U1.PH1/OSC_OUT
- new net RESET: C14.2, C6.1, D4.C, JTAG.15, S1.3, S1.4, TP7.TP, U1.NRST
- new net RTC_AF1: U1.PC13
- new net SCL: R20.2, SENSOR_I2C.3
- new net SDA: R19.2, SENSOR_I2C.4
- new net SDIO_CK: SD_CARD.5, U1.PC12
- new net SDIO_CMD: R15.1, SD_CARD.3, U1.PD2
- new net SDIO_D0: R12.1, SD_CARD.7, U1.PC8
- new net SDIO_D1: R11.1, SD_CARD.8, U1.PC9
- new net SDIO_D2: R14.1, SD_CARD.1, U1.PC10
- new net SDIO_D3: R13.1, SD_CARD.2, U1.PC11
- net +3V3: now also R11.2, R12.2, R13.2, R14.2, R15.2, S2.O, SD_CARD.4, U1.VBAT; no longer U$1.VBAT, X1.4
- net +5V: now also MICRO_USBG$2.1; no longer U$2G$2.1
- net GND: now also MICRO_USBG$1.S1, MICRO_USBG$1.S2, MICRO_USBG$1.S3, MICRO_USBG$1.S4, MICRO_USBG$2.5, R10.1, SD_CARD.6, SD_CARD.SW2, SENSOR_ADC.3, SENSOR_I2C.2, U1.VSSA, U1.VSS_3, U1.VSS_4; no longer R11.1, R12.1, R13.1, R14.1, R15.1, R5.1, U$1.VSSA, U$1.VSS_3, U$1.VSS_4, U$2G$1.S1, U$2G$1.S2, U$2G$1.S3, U$2G$1.S4, U$2G$2.5, X1.6, X1.SW2
- net N$1: now also U1.VCAP_1; no longer U$1.VCAP_1
- net N$2: now also U1.VCAP_2; no longer U$1.VCAP_2
- net VDD: now also SENSOR_ADC.1, SENSOR_I2C.1, U1.VDDA, U1.VDD_1, U1.VDD_2, U1.VDD_3, U1.VDD_4; no longer S2.O, U$1.VDDA, U$1.VDD_1, U$1.VDD_2, U$1.VDD_3, U$1.VDD_4
Other:
- note added: "ADC Sensor Block"
- note added: "BOOT0 MODE"
- note added: "BOOT1 MODE"
- note added: "Colten Nye"
- note added: "Golriz Sedaghat"
- note added: "I2C Sensor Block"
- note added: "JTAG Block"
- note added: "Open Sensor Platform Main Board"
- note added: "Power Block"
- note added: "RESET MODE"
- note added: "SD Card Block"
- note added: "Steve Peirce"
- note added: "USB Block"
- note removed: "Colten Nye, Steve Peirce, Golriz Sedaghat"
- moved on the sheet: C1, C10, C11, C12, C13, C14, C15, C2, C3, C4, C5, C6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

Commit message: Document Revision
Connections:
- net OSC_OUT renamed N$9
Other:
- moved on the sheet: C4, C5, D3, Q1, R1, R18, R19, R6, R7, R8, TP3, TP4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

Commit message: Revert "Document Revision"
This reverts commit 87a539b43a6471277175cce403c1623fabaade23.
Connections:
- net N$9 renamed OSC_OUT
Other:
- moved on the sheet: C4, C5, D3, Q1, R1, R18, R19, R6, R7, R8, TP3, TP4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
