File: Design/MainBoard_V1.2.sch (EAGLE design)
At the start: 65 parts, among them IC3 LM2936MP-3.3, Q1 25meg, Q4 2N3704, U1 STM32F20XR

Commit message: SchematicRevision
Parts:
- added LED2, LED3, LED4, LED5: (no value), led:LEDSML0805
- added MICRO_USB1, MICRO_USB2: MICRO-USB-SHIELD-ZX62R-B-5P, con-hirose:MICRO-USB-SHIELD-ZX62R-B-5P
- added Q2: 2N3704, transistor-small-signal:2N3704
- added R21: 1.5k, rcl:R-US_R0805
- added R22: 10k, rcl:R-US_R0805
- added R23: 36k, rcl:R-US_R0805
- added R24, R25, R26, R27: 0, rcl:R-US_R0805
- R16: value 10k -> 36k
- renumbered TO_BATTERY to TO_POWER_SOURCE
Connections:
- net DM renamed DM/FS
- net DP renamed DP/FS
- removed net +5V: MICRO_USBG$2.1, R17.2
- removed net RTC_AF1: U1.PC13
- new net DEBUG_LED/NP1: LED3.C
- new net DEBUG_LED/NP2: LED2.C
- new net DEBUG_LED/NP3: LED5.C
- new net DEBUG_LED/NP4: LED4.C
- new net DM/HS: MICRO_USB1G$2.2, U1.PB14
- new net DP/HS: MICRO_USB1G$2.3, R21.1, U1.PB15
- new net GPIO1: R24.1, U1.PC2
- new net GPIO2: R25.1, U1.PC1
- new net GPIO3: R26.1, U1.PB10
- new net GPIO4: R27.1, U1.PB11
- new net ID/FS: MICRO_USBG$2.4, U1.PA10
- new net ID/HS: MICRO_USB1G$2.4, U1.PB12
- new net N$11: Q2.E, R21.2
- new net N$15: Q2.B, R22.1, R23.2
- new net N$20: LED3.A, R24.2
- new net N$21: LED2.A, R25.2
- new net N$24: LED5.A, R26.2
- new net N$25: LED4.A, R27.2
- new net VBUS/FS: MICRO_USBG$2.1, R17.2, U1.PA9
- new net VBUS/HS: MICRO_USB1G$2.1, R22.2, U1.PB13
- net +3V3: now also Q2.C
- net GND: now also MICRO_USB1G$2.5, MICRO_USB2G$1.S1, MICRO_USB2G$1.S2, MICRO_USB2G$1.S3, MICRO_USB2G$1.S4, R23.1
Other:
- note added: "USB OTG FS Block"
- note added: "USB OTG HS Block"
- note removed: "USB Block"
- moved on the sheet: R19, R20, SENSOR_ADC, SENSOR_I2C
