File: Design/MainBoard_V1.3.sch (EAGLE design)
At the start: 79 parts, among them IC3 LM2936MP-3.3, Q1 25meg, Q2 2N3704, Q4 2N3704, U1 STM32F20XR

Commit message: Design Updates
Parts:
- removed D1, D3, D4, D5, D6: (no value), diode:ZENER-DIODEZD-5
- removed IC3: LM2936MP-3.3, national-semiconductor:LM2936MP-3.3
- removed JTAG: (no value), con-lstb:MA10-2
- removed LED1, LED2, LED3, LED4, LED5: (no value), led:LEDSML0805
- removed MICRO_USB, MICRO_USB1, MICRO_USB2: MICRO-USB-SHIELD-ZX62R-B-5P, con-hirose:MICRO-USB-SHIELD-ZX62R-B-5P
- removed Q1: 25meg, crystal:CRYSTALHC49S
- removed Q2, Q4: 2N3704, transistor-small-signal:2N3704
- removed R27: 0, rcl:R-US_R0805
- removed R4: 10k, rcl:R-US_R0805
- removed S2, S3, S4: (no value), SparkFun-Electromechanical:SWITCH-SPDT-SMD-A
- removed SD_CARD: SDBMF, farnell:SDBMF
- removed SENSOR_ADC, TO_POWER_SOURCE: (no value), con-lstb:MA03-1
- removed SENSOR_I2C: (no value), con-lstb:MA04-1
- removed TP1, TP3, TP4, TP5, TP6, TP7, TP8: TPB1,27, testpad:TPB1,27
- added 406C35E: 16meg, crystal:CRYSTALCTS406
- added ADC_SEN1, ADC_SEN2, ADC_SEN3, ADC_SEN4, TO_BATTERY: (no value), con-lstb:MA03-1
- added BOOT0: Boot0, SparkFun-Electromechanical:TAC_SWITCHSMD
- added C16: 4.7u, rcl:C-EUC0805
- added CURRENT_LIMITER: STMPS2141STR, SparkFun-PowerIC:V_REG_NCP1400SOT23-5
- added EJECT: Eject, SparkFun-Electromechanical:TAC_SWITCHSMD
- added G1, G2, RED, RED1: (no value), led:LEDSML0805
- added GPIOS: (no value), con-lstb:MA06-1
- added HSMS-2824-BLKG: Schottky, diode:BAS70-05
- added JP1: I2C Sensor, SparkFun-Connectors:I2C_STANDARD
- added P4SMA-4, P4SMA_1, P4SMA_2, P4SMA_3, P4SMA_4, P4SMA_5, P4SMA_6, U$1, U$2, U$3, U$4, U$5, U$6: TVS, SparkFun-DiscreteSemi:TVS
- added R28: 56, rcl:R-US_R0805
- added R29, R30: 68, rcl:R-US_R0805
- added RCLAMP0504S: (no value), microbuilder:VREG_SOT23-6_DUALAP7312
- added RESET: reset, SparkFun-Electromechanical:TAC_SWITCHSMD
- added SUPERCAP: (no value), adafruit:SUPERCAP
- added SWD_DEBUG_PORT: (no value), con-lstb:MA05-2
- added T1: NDS352AP, zetex:PMOSSOT23
- added TP11, TP14, TP15, TP16, TP17, TP18: TPB1,27, testpad:TPB1,27
- added TPS73233DBVT: 3.3V, SparkFun-PowerIC:V_REG_MIC52053.3V
- added U2: MicroSDCard, SparkFun-Connectors:USD-SOCKETNEW
- added USB_FS: MICRO-USB-SHIELD-ZX62R-B-5P, con-hirose:MICRO-USB-SHIELD-ZX62R-B-5P
- C14: value 100n -> 0.01u
- C15: value 100n -> 1u
- D2: device diode:ZENER-DIODEZD-5 -> SparkFun-DiscreteSemi:DIODESMA
- R10, R5, R7, R8: value 22 -> 10k
- R12: value 47k -> 4.7k
- R13, R14: value 47k -> 22
- R15: value 47k -> 10k
- R16: value 36k -> 47k
- R18: value 1.5k -> 10k
- R19, R20, R24, R25: value 0 -> 47k
- R21: value 1.5k -> 0
- R22: value 10k -> 47k
- R23: value 36k -> 1k
- R26: value 0 -> 56
- R6: value 22 -> 100k
- R9: value 10k -> 4.7k
- S1: value reset -> (none); device SparkFun-Electromechanical:TAC_SWITCHSMD -> SparkFun-Electromechanical:SWITCH-SPDTSMD
Connections:
- removed net +3V1: C15.1, IC3.VIN, S4.P
- removed net BOOT1: R9.1, TP9.TP, U1.PB2
- removed net DM/FS: MICRO_USBG$2.2, U1.PA11
- removed net DM/HS: MICRO_USB1G$2.2, U1.PB14
- removed net DP/FS: MICRO_USBG$2.3, R18.1, U1.PA12
- removed net DP/HS: MICRO_USB1G$2.3, R21.1, U1.PB15
- removed net ID/FS: MICRO_USBG$2.4, U1.PA10
- removed net ID/HS: MICRO_USB1G$2.4, U1.PB12
- removed net JTCK: D3.C, R7.1, TP5.TP, U1.JTCK/SWCLK/PA14
- removed net JTDI: R8.1, TP3.TP, U1.JTDI/PA15
- removed net JTDO: D5.C, R5.1, TP6.TP, U1.JTDO/TRACESSW0/PB3
- removed net JTMS: R6.1, TP4.TP, U1.JTMS/SWDIO/PA13
- removed net N$11: Q2.E, R21.2
- removed net N$12: JTAG.17, R3.2
- removed net N$19: R9.2, S3.P
- removed net N$24: LED5.A, R26.2
- removed net N$25: LED4.A, R27.2
- removed net N$33: Q4.B, R16.2, R17.1
- removed net N$8: Q4.E, R18.2
- removed net NJTRST: D6.C, JTAG.3, TP2.TP, U1.NJTRST/PB4
- removed net SCL: R20.2, SENSOR_I2C.3
- removed net SDA: R19.2, SENSOR_I2C.4
- removed net VBUS/HS: MICRO_USB1G$2.1, R22.2, U1.PB13
- removed net VDD: C10.1, C11.1, C12.1, C13.1, C3.1, C8.1, C9.1, SENSOR_ADC.1, SENSOR_I2C.1, U1.VDDA, U1.VDD_1, U1.VDD_2, U1.VDD_3, U1.VDD_4
- new net ADC1_IN0: R18.1, TP18.TP, U$6.1, U1.WKUP/PA0
- new net ADC1_IN2: ADC_SEN2.2, P4SMA_3.1, U1.PA2
- new net ADC1_IN3: ADC_SEN1.2, P4SMA_1.1, U1.PA3
- new net ADC1_IN4: ADC_SEN3.2, P4SMA-4.1, U1.PA4
- new net DEBUG_LED/NP5: GPIOS.5, R17.2
- new net DEBUG_LED/NP6: GPIOS.6, R18.2
- new net DM_IN/FS: R13.1, USB_FSG$2.2
- new net DM_OUT/FS: R13.2, RCLAMP0504S.EN1, U1.PA11
- new net DP_IN/FS: R14.1, USB_FSG$2.3
- new net DP_OUT/FS: R14.2, RCLAMP0504S.EN2, U1.PA12
- new net GPIO5: R17.1, TP17.TP, U$4.1, U1.PB12
- new net N$14: R21.1, R22.2, U2.SHIELD@2, U2.SHIELD@4
- new net N$17: G2.A, R28.2
- new net N$26: R11.1, R19.1, R20.1, R22.1, R24.1, R25.1, T1.D, U2.VCC
- new net SD_DETECT: R21.2, U1.PC5
- new net SD_EJECT: EJECT.1, EJECT.2, TP11.TP, U1.PC4
- new net SD_PWR_EN: R10.2, T1.G, U1.PA7
- new net SWCK: SWD_DEBUG_PORT.7, U1.JTCK/SWCLK/PA14
- new net SWDIO: R6.1, SWD_DEBUG_PORT.9, U1.JTMS/SWDIO/PA13
- new net TRACESWO: SWD_DEBUG_PORT.1, U1.JTDO/TRACESSW0/PB3
- new net USB/FS_OVERCURRENT: CURRENT_LIMITER.FAULT, R16.1, TP2.TP, U1.PC2
- new net USB/FS_POWERSWITCHON: CURRENT_LIMITER.EN, R15.1, U1.PB2
- new net VBAT: R23.2, SUPERCAP.+, U1.VBAT
- new net VIN: C15.1, S1.P, TPS73233DBVT.EN, TPS73233DBVT.IN
- net +3V3: now also ADC_SEN1.1, ADC_SEN2.1, ADC_SEN3.1, ADC_SEN4.1, C10.1, C11.1, C12.1, C13.1, C3.1, C8.1, C9.1, D2.A, JP1.2, R10.1, R16.2, R26.1, R28.1, R29.2, R30.2, R6.2, R9.2, SWD_DEBUG_PORT.10, T1.S, TPS73233DBVT.OUT, U1.VDDA, U1.VDD_1, U1.VDD_2, U1.VDD_3, U1.VDD_4; no longer IC3.VO, JTAG.1, JTAG.2, LED1.A, Q2.C, Q4.C, R11.2, R13.2, R14.2, S2.O, S3.O, SD_CARD.4, TP1.TP, U1.VBAT
- net ADC1_IN1: now also ADC_SEN4.2, P4SMA_2.1; no longer SENSOR_ADC.2
- net BOOT0: no longer TP8.TP
- net DEBUG_LED/NP1: now also GPIOS.1, R5.2; no longer LED3.C
- net DEBUG_LED/NP2: now also GPIOS.2, R3.2; no longer LED2.C
- net DEBUG_LED/NP3: now also GPIOS.3, R7.2; no longer LED5.C
- net DEBUG_LED/NP4: now also GPIOS.4, R8.2; no longer LED4.C
- net GND: now also ADC_SEN1.3, ADC_SEN2.3, ADC_SEN3.3, ADC_SEN4.3, BOOT0.1, BOOT0.2, C14.2, C16.2, CURRENT_LIMITER.GND, EJECT.3, EJECT.4, G1.C, JP1.1, P4SMA-4.2, P4SMA_1.2, P4SMA_2.2, P4SMA_3.2, P4SMA_4.2, P4SMA_5.2, P4SMA_6.2, RCLAMP0504S.GND, RESET.1, RESET.2, S1.O, SUPERCAP.-, SWD_DEBUG_PORT.2, SWD_DEBUG_PORT.3, SWD_DEBUG_PORT.4, SWD_DEBUG_PORT.5, SWD_DEBUG_PORT.6, SWD_DEBUG_PORT.8, TO_BATTERY.1, TO_BATTERY.2, TPS73233DBVT.GND, U$1.2, U$2.2, U$3.2, U$4.2, U$5.2, U$6.2, U2.GND, U2.SHIELD@1, U2.SHIELD@3, USB_FSG$1.S1, USB_FSG$1.S2, USB_FSG$1.S3, USB_FSG$1.S4, USB_FSG$2.5; no longer C14.1, D1.A, D2.A, D3.A, D4.A, D5.A, D6.A, IC3.GND@1, IC3.GND@2, JTAG.10, JTAG.12, JTAG.14, JTAG.16, JTAG.18, JTAG.20, JTAG.4, JTAG.6, JTAG.8, LED1.C, MICRO_USB1G$2.5, MICRO_USB2G$1.S1, MICRO_USB2G$1.S2, MICRO_USB2G$1.S3, MICRO_USB2G$1.S4, MICRO_USBG$1.S1, MICRO_USBG$1.S2, MICRO_USBG$1.S3, MICRO_USBG$1.S4, MICRO_USBG$2.5, R10.1, R16.1, R23.1, R3.1, R4.1, S1.1, S1.2, S2.S, S3.S, S4.S, SD_CARD.6, SD_CARD.SW2, SENSOR_ADC.3, SENSOR_I2C.2, TO_POWER_SOURCE.1
- net GPIO1: now also R5.1, TP9.TP, U$5.1, U1.PB14; no longer R24.1, U1.PC2
- net GPIO2: now also R3.1, TP14.TP, U$1.1, U1.PB13; no longer R25.1, U1.PC1
- net GPIO3: now also R7.1, TP15.TP, U$2.1; no longer R26.1
- net GPIO4: now also R8.1, TP16.TP, U$3.1; no longer R27.1
- net I2C1_SCL: now also JP1.4, P4SMA_4.1, R9.1; no longer R20.1
- net I2C1_SDA: now also JP1.3, P4SMA_5.1, R12.1; no longer R19.1
- net N$10: now also C14.1, TPS73233DBVT.BP; no longer JTAG.19, R4.2
- net N$13: now also RED1.C, U1.PB9; no longer JTAG.13, R5.2
- net N$15: now also D2.C, R23.1; no longer Q2.B, R22.1, R23.2
- net N$16: now also R29.1, RED.A; no longer D2.C, JTAG.7, R6.2
- net N$18: now also R30.1, RED1.A; no longer D1.C, JTAG.5, R8.2
- net N$20: now also RED.C, U1.PB8; no longer LED3.A, R24.2
- net N$21: now also HSMS-2824-BLKG.C, P4SMA_6.1, S1.S; no longer LED2.A, R25.2
- net N$3: now also G2.C, U1.PC15; no longer JTAG.9, R7.2
- net N$4: now also HSMS-2824-BLKG.A1, TO_BATTERY.3; no longer S4.O, TO_POWER_SOURCE.3
- net N$5: now also 406C35E.2; no longer Q1.1
- net N$6: now also BOOT0.3, BOOT0.4; no longer S2.P
- net N$7: now also G1.A, R26.2; no longer JTAG.11, R10.2
- net OSC_IN: now also 406C35E.1; no longer Q1.2
- net RESET: now also RESET.3, RESET.4; no longer C14.2, D4.C, JTAG.15, S1.3, S1.4, TP7.TP
- net SDIO_CK: now also U2.SCK; no longer SD_CARD.5
- net SDIO_CMD: now also R20.2, U2.DI; no longer R15.1, SD_CARD.3
- net SDIO_D0: now also R11.2, U2.DO; no longer R12.1, SD_CARD.7
- net SDIO_D1: now also R25.2, U2.RSV; no longer R11.1, SD_CARD.8
- net SDIO_D2: now also R19.2, U2.NC; no longer R14.1, SD_CARD.1
- net SDIO_D3: now also R24.2, U2.CS; no longer R13.1, SD_CARD.2
- net VBUS/FS: now also C16.1, CURRENT_LIMITER.IN, CURRENT_LIMITER.OUT, HSMS-2824-BLKG.A2, RCLAMP0504S.VIN, USB_FSG$2.1; no longer MICRO_USBG$2.1, R17.2
Other:
- note added: "BOOT0 Push Button"
- note added: "GPIO OUT"
- note added: "RESET Push Button"
- note removed: "BOOT0 MODE"
- note removed: "BOOT1 MODE"
- note removed: "GPIO Block"
- note removed: "JTAG Block"
- note removed: "RESET MODE"
- note removed: "USB OTG HS Block"
- moved on the sheet: C1, C10, C11, C12, C13, C14, C15, C2, C3, C4, C5, C6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

Commit message: Updated schematics and boards
Connections:
- net ADC1_IN1: now also ADC_SEN1.2, P4SMA_1.1, U1.PA3; no longer ADC_SEN4.2, P4SMA_2.1, U1.PA1
- net ADC1_IN3: now also ADC_SEN3.2, P4SMA-4.1, U1.PA4; no longer ADC_SEN1.2, P4SMA_1.1, U1.PA3
- net ADC1_IN4: now also ADC_SEN4.2, P4SMA_2.1, U1.PA1; no longer ADC_SEN3.2, P4SMA-4.1, U1.PA4
Changed lines of the file:
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@@
-</segment>
-</net>
-<net name="ADC1_IN1" class="0">
-<segment>
-<pinref part="U1" gate="G$1" pin="PA1"/>
-<wire x1="220.98" y1="127" x2="226.06" y2="127" width="0.1524" layer="91"/>
-<label x="226.06" y="127" size="1.778" layer="95" xref="yes"/>
-</segment>
-<segment>
-<wire x1="215.9" y1="53.34" x2="205.74" y2="53.34" width="0.1524" layer="91"/>
-<label x="203.2" y="53.34" size="1.778" layer="95" rot="R180" xref="yes"/>
-<pinref part="P4SMA_2" gate="G$1" pin="1"/>
-<wire x1="205.74" y1="53.34" x2="203.2" y2="53.34" width="0.1524" layer="91"/>
-<wire x1="205.74" y1="50.8" x2="205.74" y2="53.34" width="0.1524" layer="91"/>
-<junction x="205.74" y="53.34"/>
-<pinref part="ADC_SEN4" gate="G$1" pin="2"/>
 </segment>
 </net>
@@
 <junction x="205.74" y="25.4"/>
 <pinref part="ADC_SEN2" gate="G$1" pin="2"/>
-</segment>
-</net>
-<net name="ADC1_IN3" class="0">
-<segment>
-<pinref part="U1" gate="G$1" pin="PA3"/>
-<wire x1="220.98" y1="121.92" x2="226.06" y2="121.92" width="0.1524" layer="91"/>
-<label x="226.06" y="121.92" size="1.778" layer="95" xref="yes"/>
-</segment>
-<segment>
-<wire x1="266.7" y1="53.34" x2="256.54" y2="53.34" width="0.1524" layer="91"/>
-<label x="254" y="53.34" size="1.778" layer="95" rot="R180" xref="yes"/>
-<pinref part="P4SMA_1" gate="G$1" pin="1"/>
-<wire x1="256.54" y1="53.34" x2="254" y2="53.34" width="0.1524" layer="91"/>
-<wire x1="256.54" y1="50.8" x2="256.54" y2="53.34" width="0.1524" layer="91"/>
-<junction x="256.54" y="53.34"/>
-<pinref part="ADC_SEN1" gate="G$1" pin="2"/>
-</segment>
-</net>
-<net name="ADC1_IN4" class="0">
-<segment>
-<pinref part="U1" gate="G$1" pin="PA4"/>
-<wire x1="220.98" y1="119.38" x2="226.06" y2="119.38" width="0.1524" layer="91"/>
-<label x="226.06" y="119.38" size="1.778" layer="95" xref="yes"/>
-</segment>
-<segment>
-<wire x1="266.7" y1="25.4" x2="256.54" y2="25.4" width="0.1524" layer="91"/>
-<label x="254" y="25.4" size="1.778" layer="95" rot="R180" xref="yes"/>
-<pinref part="P4SMA-4" gate="G$1" pin="1"/>
-<wire x1="256.54" y1="25.4" x2="254" y2="25.4" width="0.1524" layer="91"/>
-<wire x1="256.54" y1="22.86" x2="256.54" y2="25.4" width="0.1524" layer="91"/>
-<junction x="256.54" y="25.4"/>
-<pinref part="ADC_SEN3" gate="G$1" pin="2"/>
 </segment>
 </net>
@@
 </segment>
 </net>
+<net name="ADC1_IN4" class="0">
+<segment>
+<wire x1="215.9" y1="53.34" x2="205.74" y2="53.34" width="0.1524" layer="91"/>
+<label x="203.2" y="53.34" size="1.778" layer="95" rot="R180" xref="yes"/>
+<pinref part="P4SMA_2" gate="G$1" pin="1"/>
+<wire x1="205.74" y1="53.34" x2="203.2" y2="53.34" width="0.1524" layer="91"/>
+<wire x1="205.74" y1="50.8" x2="205.74" y2="53.34" width="0.1524" layer="91"/>
+<junction x="205.74" y="53.34"/>
+<pinref part="ADC_SEN4" gate="G$1" pin="2"/>
+</segment>
+<segment>
+<pinref part="U1" gate="G$1" pin="PA1"/>
+<wire x1="220.98" y1="127" x2="226.06" y2="127" width="0.1524" layer="91"/>
+<label x="226.06" y="127" size="1.778" layer="95" xref="yes"/>
+</segment>
+</net>
+<net name="ADC1_IN1" class="0">
+<segment>
+<pinref part="U1" gate="G$1" pin="PA3"/>
+<wire x1="220.98" y1="121.92" x2="226.06" y2="121.92" width="0.1524" layer="91"/>
+<label x="226.06" y="121.92" size="1.778" layer="95" xref="yes"/>
+</segment>
+<segment>
+<wire x1="266.7" y1="53.34" x2="256.54" y2="53.34" width="0.1524" layer="91"/>
+<label x="254" y="53.34" size="1.778" layer="95" rot="R180" xref="yes"/>
+<pinref part="P4SMA_1" gate="G$1" pin="1"/>
+<wire x1="256.54" y1="53.34" x2="254" y2="53.34" width="0.1524" layer="91"/>
+<wire x1="256.54" y1="50.8" x2="256.54" y2="53.34" width="0.1524" layer="91"/>
+<junction x="256.54" y="53.34"/>
+<pinref part="ADC_SEN1" gate="G$1" pin="2"/>
+</segment>
+</net>
+<net name="ADC1_IN3" class="0">
+<segment>
+<pinref part="U1" gate="G$1" pin="PA4"/>
+<wire x1="220.98" y1="119.38" x2="226.06" y2="119.38" width="0.1524" layer="91"/>
+<label x="226.06" y="119.38" size="1.778" layer="95" xref="yes"/>
+</segment>
+<segment>
+<wire x1="266.7" y1="25.4" x2="256.54" y2="25.4" width="0.1524" layer="91"/>
+<label x="254" y="25.4" size="1.778" layer="95" rot="R180" xref="yes"/>
+<pinref part="P4SMA-4" gate="G$1" pin="1"/>
+<wire x1="256.54" y1="25.4" x2="254" y2="25.4" width="0.1524" layer="91"/>
+<wire x1="256.54" y1="22.86" x2="256.54" y2="25.4" width="0.1524" layer="91"/>
+<junction x="256.54" y="25.4"/>
+<pinref part="ADC_SEN3" gate="G$1" pin="2"/>
+</segment>
+</net>
