File: Design/ACC_SensorBoard.brd (EAGLE design)
At the start: 20.8 x 24.5 mm, 12 parts, among them U2 ADXL345

Commit message: Updated schematics and boards
Parts:
- removed S1: SWS001, smd-special:SMS-001
- added SW1: (no value), special:EDG-01
Connections:
- net +3V3: now also SW1.2; no longer S1.2
- net GND: now also SW1.1; no longer S1.1
Routing:
- net +3V3: track 90.7 -> 103.2 mm, vias 3 -> 4
- net GND: track 74.9 -> 64.9 mm
Changed lines of the file:
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@@
 <attribute name="VALUE" x="0.0508" y="12.827" size="1.27" layer="27" rot="R270"/>
 </element>
-<element name="S1" library="smd-special" package="SMS-001" value="SWS001" x="10.5156" y="21.8948" smashed="yes" rot="R90"/>
+<element name="SW1" library="special" package="EDG-01" value="" x="10.2108" y="22.0218" smashed="yes" rot="R270">
+<attribute name="VALUE" x="3.6068" y="23.9268" size="1.27" layer="27" ratio="10" rot="R270"/>
+</element>
 </elements>
 <signals>
@@
 <vertex x="0" y="0"/>
 </polygon>
-<contactref element="S1" pad="1"/>
 <wire x1="9.183521875" y1="11.75021875" x2="9.183521875" y2="12.762078125" width="0.4064" layer="1"/>
 <wire x1="9.183521875" y1="12.762078125" x2="9.144" y2="12.8016" width="0.4064" layer="1"/>
@@
 <wire x1="15.0876" y1="4.191" x2="12.5476" y2="4.191" width="0.4064" layer="1"/>
 <wire x1="12.5476" y1="4.191" x2="11.557" y2="3.2004" width="0.4064" layer="1"/>
-<wire x1="15.0114" y1="21.8948" x2="19.177" y2="21.8948" width="0.4064" layer="1"/>
-<wire x1="19.177" y1="21.8948" x2="19.431" y2="21.6408" width="0.4064" layer="1"/>
-<wire x1="19.431" y1="21.6408" x2="19.431" y2="14.6304" width="0.4064" layer="1"/>
-<wire x1="19.431" y1="14.6304" x2="19.3548" y2="14.5542" width="0.4064" layer="1"/>
-<wire x1="19.3548" y1="14.5542" x2="17.356984375" y2="14.5542" width="0.4064" layer="1"/>
-<wire x1="17.356984375" y1="14.5542" x2="17.305021875" y2="14.5022375" width="0.4064" layer="1"/>
 <wire x1="17.305021875" y1="14.5022375" x2="17.305021875" y2="11.701778125" width="0.4064" layer="1"/>
 <wire x1="17.305021875" y1="11.701778125" x2="17.4244" y2="11.5824" width="0.4064" layer="1"/>
@@
 <wire x1="5.4864" y1="19.2786" x2="5.4864" y2="14.7828" width="0.4064" layer="1"/>
 <wire x1="5.4864" y1="14.7828" x2="5.334" y2="14.6304" width="0.4064" layer="1"/>
+<contactref element="SW1" pad="1"/>
+<wire x1="6.4008" y1="22.0218" x2="5.4864" y2="22.0218" width="0.4064" layer="16"/>
+<wire x1="5.4864" y1="22.0218" x2="5.4864" y2="19.2786" width="0.4064" layer="16"/>
 </signal>
 <signal name="SDA_ACC">
@@
 <contactref element="M2" pad="2"/>
 <contactref element="F2" pad="2"/>
-<contactref element="S1" pad="2"/>
 <contactref element="U2" pad="12"/>
 <wire x1="11.583521875" y1="9.55021875" x2="11.583521875" y2="6.75278125" width="0.4064" layer="1"/>
@@
 <wire x1="11.5824" y1="10.5918" x2="11.5824" y2="9.551340625" width="0.254" layer="1"/>
 <wire x1="11.5824" y1="9.551340625" x2="11.583521875" y2="9.55021875" width="0.254" layer="1"/>
-<wire x1="6.0198" y1="21.8948" x2="4.2418" y2="21.8948" width="0.4064" layer="1"/>
 <wire x1="4.2418" y1="21.8948" x2="4.191" y2="21.9456" width="0.4064" layer="1"/>
 <via x="4.191" y="21.9456" extent="1-16" drill="0.6" diameter="0.254"/>
@@
 <wire x1="19.2786" y1="9.0678" x2="17.4498" y2="9.0678" width="0.4064" layer="16"/>
 <wire x1="17.4498" y1="9.0678" x2="17.4244" y2="9.0424" width="0.4064" layer="16"/>
+<contactref element="SW1" pad="2"/>
+<wire x1="14.0208" y1="22.0218" x2="19.431" y2="22.0218" width="0.4064" layer="1"/>
+<wire x1="19.431" y1="22.0218" x2="19.431" y2="15.621" width="0.4064" layer="1"/>
+<via x="19.431" y="15.621" extent="1-16" drill="0.5" diameter="0.254"/>
+<wire x1="19.431" y1="15.621" x2="19.431" y2="13.2588" width="0.4064" layer="16"/>
+<wire x1="19.431" y1="13.2588" x2="19.3548" y2="13.1826" width="0.4064" layer="16"/>
 </signal>
 <signal name="N$15">

Commit message: Design Final Revision
Parts:
- removed U$2: TVS, SparkFun-DiscreteSemi:SMA-DIODE
- added GND: TVS, SparkFun-DiscreteSemi:SMA-DIODE
- moved M2 1.27 mm to (18.7, 10.3)
- moved M1 1.27 mm to (4.50, 10.3)
- moved R2 1.27 mm to (5.09, 4.37)
- moved C1 1.27 mm to (18.8, 4.06)
- moved C2 1.27 mm to (12.0, 6.65)
- moved F1 1.27 mm to (12.9, 17.4)
- moved F2 1.27 mm to (12.8, 3.20)
- moved R1 1.27 mm to (11.9, 14.3)
- moved SW1 1.27 mm to (11.5, 22.0)
- moved U$1 1.27 mm to (18.6, 16.7)
- moved U2 1.27 mm to (11.7, 10.7)
Connections:
- net GND: now also GND.A; no longer U$2.A
- net SCL_ACC: now also GND.C; no longer U$2.C
Routing:
- net +3V3: track 103.2 -> 78.5 mm, vias 4 -> 2
- net GND: vias 2 -> 20
Other:
- board size 20.8 x 24.5 mm -> 23.3 x 24.5 mm

Commit message: Updating/Cleaning-up documents
Parts:
- removed GND, U$1: TVS, SparkFun-DiscreteSemi:SMA-DIODE
- removed SW1: (no value), special:EDG-01
- added S1: (no value), SparkFun-Electromechanical:AYZ0202
- moved R2 12.6 mm to (6.10, 16.9), turned to 180 degrees
- moved R1 0.92 mm to (12.4, 15.0)
- moved C1 0.72 mm to (19.3, 4.57)
- moved F1 0.72 mm to (13.4, 17.9)
- moved F2 0.72 mm to (13.3, 3.71)
- moved U2 0.72 mm to (12.2, 11.2)
- moved C2 0.72 mm to (12.5, 7.16)
- moved M1 0.72 mm to (5.00, 10.8)
- moved M2 0.72 mm to (19.2, 10.8)
Connections:
- new net N$1: S1.2, U2.12
- net +3V3: now also S1.1; no longer SW1.2, U2.12
- net GND: now also S1.3; no longer GND.A, SW1.1, U$1.A
- net SCL_ACC: no longer GND.C
- net SDA_ACC: no longer U$1.C
Routing:
- net SCL_ACC: track 60.6 -> 38.9 mm, vias 4 -> 2
- net GND: track 64.9 -> 52.1 mm, vias 20 -> 5
- net N$1: track 0.00 -> 11.1 mm
- net SDA_ACC: track 32.4 -> 27.2 mm
- net +3V3: track 78.5 -> 83.4 mm, vias 2 -> 3
Other:
- board size 23.3 x 24.5 mm -> 23.8 x 22 mm
