File: Design/ACC_SensorBoard.sch (EAGLE design)
At the start: 12 parts, among them U2 ADXL345

Commit message: Updated schematics and boards
Parts:
- removed S1: SWS001, smd-special:SWS001
- added SW1: (no value), special:SW_DIP-1
Connections:
- net +3V3: now also SW1.2; no longer S1.2
- net GND: now also SW1.1; no longer S1.1
Changed lines of the file:
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@@
 <part name="M2" library="pinhead" deviceset="PINHD-1X2" device=""/>
 <part name="M1" library="pinhead" deviceset="PINHD-1X2" device=""/>
-<part name="S1" library="smd-special" deviceset="SWS001" device=""/>
 <part name="SUPPLY6" library="supply2" deviceset="GND" device=""/>
+<part name="SW1" library="special" deviceset="SW_DIP-1" device=""/>
 </parts>
 <sheets>
@@
 <instance part="M2" gate="G$1" x="177.8" y="88.9" rot="R180"/>
 <instance part="M1" gate="G$1" x="177.8" y="99.06" rot="R180"/>
-<instance part="S1" gate="G$1" x="134.62" y="78.74"/>
-<instance part="SUPPLY6" gate="GND" x="134.62" y="71.12"/>
+<instance part="SUPPLY6" gate="GND" x="134.62" y="66.04"/>
+<instance part="SW1" gate="G$1" x="134.62" y="78.74" rot="R270"/>
 </instances>
 <busses>
@@
 </segment>
 <segment>
-<pinref part="S1" gate="G$1" pin="1"/>
+<pinref part="SW1" gate="G$1" pin="1"/>
 <pinref part="SUPPLY6" gate="GND" pin="GND"/>
+<wire x1="134.62" y1="68.58" x2="134.62" y2="71.12" width="0.1524" layer="91"/>
 </segment>
 </net>
@@
 <junction x="134.62" y="109.22"/>
 <pinref part="U2" gate="G$1" pin="SDO"/>
-<pinref part="S1" gate="G$1" pin="2"/>
 <wire x1="127" y1="93.98" x2="134.62" y2="93.98" width="0.1524" layer="91"/>
 <wire x1="134.62" y1="93.98" x2="134.62" y2="86.36" width="0.1524" layer="91"/>
 <junction x="134.62" y="93.98"/>
 <wire x1="134.62" y1="93.98" x2="134.62" y2="109.22" width="0.1524" layer="91"/>
+<pinref part="SW1" gate="G$1" pin="2"/>
 </segment>
 <segment>

Commit message: Design Final Revision
Parts:
- renumbered U$2 to GND
Changed lines of the file:
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@@
 <part name="R2" library="rcl" deviceset="R-US_" device="R0805" value="4.7k"/>
 <part name="U$1" library="SparkFun-DiscreteSemi" deviceset="TVS" device=""/>
-<part name="U$2" library="SparkFun-DiscreteSemi" deviceset="TVS" device=""/>
+<part name="GND" library="SparkFun-DiscreteSemi" deviceset="TVS" device=""/>
 <part name="SUPPLY3" library="supply2" deviceset="GND" device=""/>
 <part name="SUPPLY4" library="supply2" deviceset="GND" device=""/>
@@
 <instance part="R2" gate="G$1" x="157.48" y="101.6" rot="R270"/>
 <instance part="U$1" gate="G$1" x="147.32" y="81.28" rot="R90"/>
-<instance part="U$2" gate="G$1" x="154.94" y="73.66" rot="R90"/>
+<instance part="GND" gate="G$1" x="154.94" y="73.66" rot="R90"/>
 <instance part="SUPPLY3" gate="GND" x="147.32" y="76.2"/>
 <instance part="SUPPLY4" gate="GND" x="154.94" y="68.58"/>
@@
 </segment>
 <segment>
-<pinref part="U$2" gate="G$1" pin="1"/>
+<pinref part="GND" gate="G$1" pin="1"/>
 <pinref part="SUPPLY4" gate="GND" pin="GND"/>
 </segment>
@@
 <label x="157.48" y="88.9" size="1.778" layer="95" xref="yes"/>
 <pinref part="R2" gate="G$1" pin="2"/>
-<pinref part="U$2" gate="G$1" pin="2"/>
+<pinref part="GND" gate="G$1" pin="2"/>
 <wire x1="154.94" y1="78.74" x2="154.94" y2="88.9" width="0.1524" layer="91"/>
 <junction x="154.94" y="88.9"/>

Commit message: Updating/Cleaning-up documents
Parts:
- removed GND, U$1: TVS, SparkFun-DiscreteSemi:TVS
- removed SW1: (no value), special:SW_DIP-1
- added S1: (no value), SparkFun-Electromechanical:SWITCH-SPDTSMD
Connections:
- new net N$1: S1.P, U2.SDO
- net +3V3: now also S1.O; no longer SW1.2, U2.SDO
- net GND: now also S1.S; no longer GND.1, SW1.1, U$1.1
- net SCL_ACC: no longer GND.2
- net SDA_ACC: no longer U$1.2
Changed lines of the file:
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@@
 <part name="R1" library="rcl" deviceset="R-US_" device="R0805" value="4.7k"/>
 <part name="R2" library="rcl" deviceset="R-US_" device="R0805" value="4.7k"/>
-<part name="U$1" library="SparkFun-DiscreteSemi" deviceset="TVS" device=""/>
-<part name="GND" library="SparkFun-DiscreteSemi" deviceset="TVS" device=""/>
-<part name="SUPPLY3" library="supply2" deviceset="GND" device=""/>
-<part name="SUPPLY4" library="supply2" deviceset="GND" device=""/>
 <part name="SUPPLY1" library="supply2" deviceset="GND" device=""/>
 <part name="C2" library="rcl" deviceset="C-US" device="C0805" value="0.1u"/>
@@
 <part name="M1" library="pinhead" deviceset="PINHD-1X2" device=""/>
 <part name="SUPPLY6" library="supply2" deviceset="GND" device=""/>
-<part name="SW1" library="special" deviceset="SW_DIP-1" device=""/>
+<part name="S1" library="SparkFun-Electromechanical" deviceset="SWITCH-SPDT" device="SMD"/>
 </parts>
 <sheets>
@@
 <instance part="R1" gate="G$1" x="149.86" y="101.6" rot="R270"/>
 <instance part="R2" gate="G$1" x="157.48" y="101.6" rot="R270"/>
-<instance part="U$1" gate="G$1" x="147.32" y="81.28" rot="R90"/>
-<instance part="GND" gate="G$1" x="154.94" y="73.66" rot="R90"/>
-<instance part="SUPPLY3" gate="GND" x="147.32" y="76.2"/>
-<instance part="SUPPLY4" gate="GND" x="154.94" y="68.58"/>
 <instance part="SUPPLY1" gate="GND" x="198.12" y="78.74"/>
 <instance part="C2" gate="G$1" x="83.82" y="91.44"/>
@@
 <instance part="M2" gate="G$1" x="177.8" y="88.9" rot="R180"/>
 <instance part="M1" gate="G$1" x="177.8" y="99.06" rot="R180"/>
-<instance part="SUPPLY6" gate="GND" x="134.62" y="66.04"/>
-<instance part="SW1" gate="G$1" x="134.62" y="78.74" rot="R270"/>
+<instance part="SUPPLY6" gate="GND" x="142.24" y="73.66"/>
+<instance part="S1" gate="1" x="134.62" y="81.28"/>
 </instances>
 <busses>
@@
 </segment>
 <segment>
-<pinref part="U$1" gate="G$1" pin="1"/>
-<pinref part="SUPPLY3" gate="GND" pin="GND"/>
-</segment>
-<segment>
-<pinref part="GND" gate="G$1" pin="1"/>
-<pinref part="SUPPLY4" gate="GND" pin="GND"/>
-</segment>
-<segment>
 <wire x1="180.34" y1="86.36" x2="193.04" y2="86.36" width="0.1524" layer="91"/>
 <wire x1="193.04" y1="86.36" x2="198.12" y2="86.36" width="0.1524" layer="91"/>
@@
 </segment>
 <segment>
-<pinref part="SW1" gate="G$1" pin="1"/>
 <pinref part="SUPPLY6" gate="GND" pin="GND"/>
-<wire x1="134.62" y1="68.58" x2="134.62" y2="71.12" width="0.1524" layer="91"/>
+<wire x1="142.24" y1="76.2" x2="142.24" y2="78.74" width="0.1524" layer="91"/>
+<pinref part="S1" gate="1" pin="S"/>
+<wire x1="139.7" y1="78.74" x2="142.24" y2="78.74" width="0.1524" layer="91"/>
 </segment>
 </net>
@@
 <segment>
 <pinref part="U2" gate="G$1" pin="SDA"/>
-<wire x1="127" y1="91.44" x2="147.32" y2="91.44" width="0.1524" layer="91"/>
-<wire x1="147.32" y1="91.44" x2="149.86" y2="91.44" width="0.1524" layer="91"/>
+<wire x1="127" y1="91.44" x2="149.86" y2="91.44" width="0.1524" layer="91"/>
 <wire x1="149.86" y1="91.44" x2="149.86" y2="96.52" width="0.1524" layer="91"/>
 <label x="149.86" y="91.44" size="1.778" layer="95" xref="yes"/>
 <pinref part="R1" gate="G$1" pin="2"/>
-<pinref part="U$1" gate="G$1" pin="2"/>
-<wire x1="147.32" y1="86.36" x2="147.32" y2="91.44" width="0.1524" layer="91"/>
-<junction x="147.32" y="91.44"/>
 </segment>
 <segment>
@@
 <segment>
 <pinref part="U2" gate="G$1" pin="SCL"/>
-<wire x1="127" y1="88.9" x2="154.94" y2="88.9" width="0.1524" layer="91"/>
-<wire x1="154.94" y1="88.9" x2="157.48" y2="88.9" width="0.1524" layer="91"/>
+<wire x1="127" y1="88.9" x2="157.48" y2="88.9" width="0.1524" layer="91"/>
 <wire x1="157.48" y1="88.9" x2="157.48" y2="96.52" width="0.1524" layer="91"/>
 <label x="157.48" y="88.9" size="1.778" layer="95" xref="yes"/>
 <pinref part="R2" gate="G$1" pin="2"/>
-<pinref part="GND" gate="G$1" pin="2"/>
-<wire x1="154.94" y1="78.74" x2="154.94" y2="88.9" width="0.1524" layer="91"/>
-<junction x="154.94" y="88.9"/>
 </segment>
 <segment>
@@
 <wire x1="129.54" y1="109.22" x2="129.54" y2="111.76" width="0.1524" layer="91"/>
 <wire x1="149.86" y1="106.68" x2="149.86" y2="109.22" width="0.1524" layer="91"/>
-<wire x1="149.86" y1="109.22" x2="134.62" y2="109.22" width="0.1524" layer="91"/>
+<wire x1="149.86" y1="109.22" x2="142.24" y2="109.22" width="0.1524" layer="91"/>
 <pinref part="R2" gate="G$1" pin="1"/>
-<wire x1="134.62" y1="109.22" x2="129.54" y2="109.22" width="0.1524" layer="91"/>
+<wire x1="142.24" y1="109.22" x2="129.54" y2="109.22" width="0.1524" layer="91"/>
 <wire x1="157.48" y1="106.68" x2="157.48" y2="109.22" width="0.1524" layer="91"/>
 <wire x1="157.48" y1="109.22" x2="149.86" y2="109.22" width="0.1524" layer="91"/>
 <junction x="149.86" y="109.22"/>
 <junction x="129.54" y="109.22"/>
-<junction x="134.62" y="109.22"/>
-<pinref part="U2" gate="G$1" pin="SDO"/>
-<wire x1="127" y1="93.98" x2="134.62" y2="93.98" width="0.1524" layer="91"/>
-<wire x1="134.62" y1="93.98" x2="134.62" y2="86.36" width="0.1524" layer="91"/>
-<junction x="134.62" y="93.98"/>
-<wire x1="134.62" y1="93.98" x2="134.62" y2="109.22" width="0.1524" layer="91"/>
-<pinref part="SW1" gate="G$1" pin="2"/>
+<pinref part="S1" gate="1" pin="O"/>
+<wire x1="139.7" y1="83.82" x2="142.24" y2="83.82" width="0.1524" layer="91"/>
+<wire x1="142.24" y1="83.82" x2="142.24" y2="109.22" width="0.1524" layer="91"/>
+<junction x="142.24" y="109.22"/>
 </segment>
 <segment>
@@
 </segment>
 </net>
+<net name="N$1" class="0">
+<segment>
+<pinref part="S1" gate="1" pin="P"/>
+<wire x1="132.08" y1="81.28" x2="129.54" y2="81.28" width="0.1524" layer="91"/>
+<wire x1="129.54" y1="81.28" x2="129.54" y2="93.98" width="0.1524" layer="91"/>
+<pinref part="U2" gate="G$1" pin="SDO"/>
+<wire x1="129.54" y1="93.98" x2="127" y2="93.98" width="0.1524" layer="91"/>
+</segment>
+</net>
