File: Design/MainBoardV2.sch (EAGLE design)
At the start: 92 parts, among them P4SMA-4 TVS, P4SMA_1 TVS, P4SMA_2 TVS, P4SMA_3 TVS, P4SMA_4 TVS, P4SMA_5 TVS, P4SMA_6 TVS, T1 NDS352AP, U1 STM32F20XR, U2 MicroSDCard

Commit message: 2nd Version of Board and Schematic
Parts:
- removed CURRENT_LIMITER: STMPS2141STR, SparkFun-PowerIC:V_REG_NCP1400SOT23-5
- removed G1: (no value), led:LEDSML0805
- removed P4SMA-4, P4SMA_1, P4SMA_2, P4SMA_3, P4SMA_4, P4SMA_5, P4SMA_6, U$1, U$2, U$3, U$4, U$5, U$6: TVS, SparkFun-DiscreteSemi:TVS
- added C17: 100n, rcl:C-EUC0805
- added C18, C19: 47p, rcl:C-EUC0805
- added C20: 10n, rcl:C-EUC0805
- added IC1: FT230XS, ftdichip:FT230XS
- added R27, R31, R32, R33: 10k, rcl:R-US_R0805
- added R34: 1k, rcl:R-US_R0805
- added R4: 22, rcl:R-US_R0805
- added STMPS2141STR: (no value), microbuilder:NCP1400A_STEPUP
- added TP1, TP3, TP4, TP5: TPB1,27, testpad:TPB1,27
- added TVS1, TVS10, TVS11, TVS13, TVS14, TVS15, TVS16, TVS17, TVS2, TVS3, TVS4, TVS5, TVS6, TVS7, TVS8, TVS9: TVS, SparkFun-DiscreteSemi:TVS
- added TVS12: P4SMA, SparkFun-DiscreteSemi:TVS
- C4, C5: value 22p -> 20p
- R1: value 904.3 -> 1k
- R13, R14: value 22 -> 27
- R26: value 56 -> 22
- R28: value 56 -> 1k
- R29, R30: value 68 -> 1k
- RCLAMP0504S: device microbuilder:VREG_SOT23-6_DUALAP7312 -> microbuilder:BREAKOUT_SOT23-6
- SWD_DEBUG_PORT: device con-lstb:MA05-2 -> microbuilder:JTAG-CORTEXM3
- renumbered G2 to GREEN, RED1 to BLUE
Connections:
- net N$9 renamed OSC_OUT
- removed net ADC1_IN1: ADC_SEN1.2, P4SMA_1.1, U1.PA3
- removed net ADC1_IN2: ADC_SEN2.2, P4SMA_3.1, U1.PA2
- removed net ADC1_IN3: ADC_SEN3.2, P4SMA-4.1, U1.PA4
- removed net ADC1_IN4: ADC_SEN4.2, P4SMA_2.1, U1.PA1
- new net BLUE: ADC_SEN1.2, TVS7.1, U1.PA3
- new net GREEN: ADC_SEN3.2, TVS8.1, U1.PA4
- new net N$11: BOOT0.1, BOOT0.2, R34.1
- new net N$8: IC1.USBDM, R14.2
- new net N$9: IC1.USBDP, R13.1
- new net PINK: ADC_SEN2.2, TVS10.1, U1.PA2
- new net RED: ADC_SEN4.2, TVS9.1, U1.PA1
- new net USART3_CTS: IC1.!CTS, R27.1, TVS14.1, U1.PB13
- new net USART3_RTS: IC1.!RTS, R32.1, TVS17.1, U1.PB14
- new net USART3_RX: IC1.RXD, R31.1, TVS15.1, U1.PB11
- new net USART3_TX: IC1.TXD, R33.1, TVS16.1, U1.PB10
- new net VBUS/FS_IN: STMPS2141STR.IN, USB_FSG$2.1
- net +3V3: now also R27.2, R31.2, R32.2, R33.2, R34.2, SWD_DEBUG_PORT.1; no longer R26.1, SWD_DEBUG_PORT.10
- net ADC1_IN0: now also TVS6.1; no longer U$6.1
- net DM_IN/FS: now also R4.1; no longer R13.1
- net DM_OUT/FS: now also C19.1, R14.1, R4.2, RCLAMP0504S.4; no longer R13.2, RCLAMP0504S.EN1
- net DP_IN/FS: now also R26.1; no longer R14.1
- net DP_OUT/FS: now also C18.1, R13.2, R26.2, RCLAMP0504S.3; no longer R14.2, RCLAMP0504S.EN2
- net GND: now also C17.2, C18.2, C19.2, C20.2, IC1.GND, IC1.GND@1, RCLAMP0504S.2, STMPS2141STR.GND, SWD_DEBUG_PORT.9, TVS1.2, TVS10.2, TVS11.2, TVS12.2, TVS13.2, TVS14.2, TVS15.2, TVS16.2, TVS17.2, TVS2.2, TVS3.2, TVS4.2, TVS5.2, TVS6.2, TVS7.2, TVS8.2, TVS9.2; no longer BOOT0.1, BOOT0.2, CURRENT_LIMITER.GND, G1.C, P4SMA-4.2, P4SMA_1.2, P4SMA_2.2, P4SMA_3.2, P4SMA_4.2, P4SMA_5.2, P4SMA_6.2, RCLAMP0504S.GND, SWD_DEBUG_PORT.2, SWD_DEBUG_PORT.4, SWD_DEBUG_PORT.6, SWD_DEBUG_PORT.8, U$1.2, U$2.2, U$3.2, U$4.2, U$5.2, U$6.2
- net GPIO1: now also TVS1.1, U1.PB2; no longer U$5.1, U1.PB14
- net GPIO2: now also TVS2.1, U1.PB0; no longer U$1.1, U1.PB13
- net GPIO3: now also TVS3.1, U1.PB1; no longer U$2.1, U1.PB10
- net GPIO4: now also TVS4.1, U1.PC13; no longer U$3.1, U1.PB11
- net GPIO5: now also TVS5.1, U1.PC14; no longer U$4.1, U1.PB12
- net I2C1_SCL: now also TVS12.1; no longer P4SMA_4.1
- net I2C1_SDA: now also TVS11.1; no longer P4SMA_5.1
- net N$21: now also TVS13.1; no longer P4SMA_6.1
- net N$7: now also C17.1, IC1.!RESET, IC1.3V3OUT, IC1.VCCIO; no longer G1.A, R26.2
- net RESET: now also SWD_DEBUG_PORT.10, TP4.TP
- net SWCK: now also SWD_DEBUG_PORT.4, TP3.TP; no longer SWD_DEBUG_PORT.7
- net SWDIO: now also SWD_DEBUG_PORT.2, TP1.TP; no longer SWD_DEBUG_PORT.9
- net TRACESWO: now also SWD_DEBUG_PORT.6, TP5.TP; no longer SWD_DEBUG_PORT.1
- net USB/FS_OVERCURRENT: now also STMPS2141STR.FAULT; no longer CURRENT_LIMITER.FAULT
- net USB/FS_POWERSWITCHON: now also STMPS2141STR.EN, U1.PB5; no longer CURRENT_LIMITER.EN, U1.PB2
- net VBUS/FS: now also C20.1, IC1.VCC, RCLAMP0504S.5, STMPS2141STR.OUT; no longer CURRENT_LIMITER.IN, CURRENT_LIMITER.OUT, RCLAMP0504S.VIN, USB_FSG$2.1
Other:
- note added: "TVS array protection for USB data lines"
- note added: "USB Power Protection"
- note added: "USB to UART Converter Block"
- note removed: "BOOT0 Push Button"
- note removed: "RESET Push Button"
- moved on the sheet: ADC_SEN1, ADC_SEN2, ADC_SEN3, ADC_SEN4, BOOT0, C14, C15, C16, C6, C7, EJECT, GPIOS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

Commit message: Modified revision of board and schematic
Parts:
- removed ADC_SEN4: (no value), con-lstb:MA03-1
- removed TP11, TP5: TPB1,27, testpad:TPB1,27
- removed TVS14, TVS15, TVS16, TVS17, TVS8: TVS, SparkFun-DiscreteSemi:TVS
- added C21: 10u, rcl:C-EUC0805
- added PROGRAM: Program, SparkFun-Electromechanical:TAC_SWITCHSMD
- added RXLED, TXLED: (no value), led:LEDSML0805
- added USBTOUART: USB_Shield, con-hirose:MICRO-USB-SHIELD-ZX62R-B-5P
- R27, R32: value 10k -> 1k
- USB_FS: value MICRO-USB-SHIELD-ZX62R-B-5P -> USB_Shield
- renumbered RCLAMP0504S to RCLAMP, STMPS2141STR to 2141, TPS73233DBVT to TPS73233
Connections:
- removed net ADC1_IN0: R18.1, TP18.TP, TVS6.1, U1.WKUP/PA0
- removed net PINK: ADC_SEN2.2, TVS10.1, U1.PA2
- removed net TRACESWO: SWD_DEBUG_PORT.6, TP5.TP, U1.JTDO/TRACESSW0/PB3
- removed net USART3_CTS: IC1.!CTS, R27.1, TVS14.1, U1.PB13
- removed net USART3_RTS: IC1.!RTS, R32.1, TVS17.1, U1.PB14
- new net DM: C19.1, R14.1, USBTOUARTG$2.2
- new net DP: C18.1, R13.2, USBTOUARTG$2.3
- new net GPIO6: R18.1, TP18.TP, TVS6.1, U1.PB14
- new net N$12: R27.2, TXLED.A
- new net N$19: R32.1, RXLED.A
- new net N$22: IC1.CBUS1, RXLED.C
- new net N$23: IC1.CBUS2, TXLED.C
- new net PROGRAMMING_EN: PROGRAM.1, PROGRAM.2, U1.PB12
- net +3V3: now also R27.1; no longer ADC_SEN4.1, R27.2
- net DM_OUT/FS: no longer C19.1, R14.1
- net DP_OUT/FS: no longer C18.1, R13.2
- net GND: now also C21.2, PROGRAM.3, PROGRAM.4, USBTOUARTG$1.S1, USBTOUARTG$1.S2, USBTOUARTG$1.S3, USBTOUARTG$1.S4, USBTOUARTG$2.5; no longer ADC_SEN4.3, TVS14.2, TVS15.2, TVS16.2, TVS17.2, TVS8.2
- net GPIO1: now also U1.PA6; no longer U1.PB2
- net GPIO2: now also U1.PA8; no longer U1.PB0
- net GPIO3: now also U1.PA10; no longer U1.PB1
- net GPIO4: now also U1.PC0; no longer U1.PC13
- net GPIO5: now also U1.PB13; no longer U1.PC14
- net GREEN: now also ADC_SEN2.2, TVS10.1, U1.PA2; no longer ADC_SEN3.2, TVS8.1, U1.PA4
- net RED: now also ADC_SEN3.2; no longer ADC_SEN4.2
- net SD_EJECT: no longer TP11.TP
- net USART3_RX: now also U1.PB10; no longer TVS15.1, U1.PB11
- net USART3_TX: now also U1.PB11; no longer TVS16.1, U1.PB10
- net VBUS/FS_IN: now also C21.1, USBTOUARTG$2.1
Other:
- note added: "ADC Sensor Headers"
- note added: "I2C Sensor Header"
- note added: "USB To UART"
- note removed: "ADC Sensor Block"
- note removed: "I2C Sensor Block"
- moved on the sheet: ADC_SEN1, ADC_SEN2, ADC_SEN3, C17, GPIOS, R15, R17, R18, R27, R3, R32, R5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

Commit message: Updating/Cleaning-up documents
Connections:
- net GND: no longer TO_BATTERY.2
- net VBUS/FS: now also TO_BATTERY.2
Changed lines of the file:
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@@
 <pinref part="TO_BATTERY" gate="G$1" pin="1"/>
 <wire x1="25.4" y1="55.88" x2="27.94" y2="55.88" width="0.1524" layer="91"/>
-<pinref part="TO_BATTERY" gate="G$1" pin="2"/>
-<wire x1="25.4" y1="58.42" x2="27.94" y2="58.42" width="0.1524" layer="91"/>
-<wire x1="27.94" y1="58.42" x2="27.94" y2="55.88" width="0.1524" layer="91"/>
 <pinref part="SUPPLY23" gate="GND" pin="GND"/>
 <wire x1="27.94" y1="53.34" x2="27.94" y2="55.88" width="0.1524" layer="91"/>
-<junction x="27.94" y="55.88"/>
 </segment>
 <segment>
@@
 <pinref part="U1" gate="G$1" pin="PA12"/>
 <wire x1="220.98" y1="99.06" x2="226.06" y2="99.06" width="0.1524" layer="91"/>
-<label x="226.06" y="99.06" size="1.4224" layer="95" xref="yes"/>
+<label x="226.06" y="99.06" size="1.27" layer="95" xref="yes"/>
 </segment>
 <segment>
@@
 <pinref part="HSMS-2824-BLKG" gate="G$1" pin="A2"/>
 <wire x1="35.56" y1="48.26" x2="35.56" y2="43.18" width="0.1524" layer="91"/>
-<wire x1="35.56" y1="43.18" x2="27.94" y2="43.18" width="0.1524" layer="91"/>
-</segment>
-<segment>
+<wire x1="35.56" y1="43.18" x2="33.02" y2="43.18" width="0.1524" layer="91"/>
+<pinref part="TO_BATTERY" gate="G$1" pin="2"/>
+<wire x1="33.02" y1="43.18" x2="27.94" y2="43.18" width="0.1524" layer="91"/>
+<wire x1="25.4" y1="58.42" x2="33.02" y2="58.42" width="0.1524" layer="91"/>
+<wire x1="33.02" y1="58.42" x2="33.02" y2="43.18" width="0.1524" layer="91"/>
+<junction x="33.02" y="43.18"/>
+</segment>
+<segment>
