File: Design/VOC_SensorBoard.brd (EAGLE design)
At the start: 20.1 x 20.3 mm, 4 parts

Commit message: Design Final Revision
Routing:
- net GND: vias 0 -> 21
Other:
- board text added: "VOC Sensor Board"
- board text removed: "VOC Sensor Board V.1"
Changed lines of the file:
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@@
 <wire x1="20.0714" y1="20.292259375" x2="0" y2="20.292259375" width="0" layer="20"/>
 <wire x1="0" y1="20.292259375" x2="0" y2="0" width="0" layer="20"/>
-<text x="0.66801875" y="18.521678125" size="0.6096" layer="25">VOC Sensor Board V.1</text>
+<text x="0.66801875" y="18.521678125" size="0.6096" layer="25">VOC Sensor Board </text>
 <text x="0.66548125" y="17.0053" size="0.6096" layer="25">Colten Nye, Steve Peirce, Golriz Sedaghat</text>
 </plain>
@@
 <vertex x="0" y="0"/>
 </polygon>
+<via x="1.4986" y="18.3896" extent="1-16" drill="0.5" diameter="0.254"/>
+<via x="4.445" y="14.8844" extent="1-16" drill="0.6"/>
+<via x="2.5908" y="11.7348" extent="1-16" drill="0.6"/>
+<via x="5.5626" y="8.2042" extent="1-16" drill="0.6"/>
+<via x="4.1148" y="3.7846" extent="1-16" drill="0.6"/>
+<via x="2.4384" y="1.2192" extent="1-16" drill="0.5" diameter="0.254"/>
+<via x="14.7066" y="1.3462" extent="1-16" drill="0.5" diameter="0.254"/>
+<via x="14.5288" y="4.5466" extent="1-16" drill="0.6"/>
+<via x="18.0848" y="2.1844" extent="1-16" drill="0.5" diameter="0.254"/>
+<via x="18.9992" y="9.6012" extent="1-16" drill="0.5" diameter="0.254"/>
+<via x="14.224" y="9.5758" extent="1-16" drill="0.6"/>
+<via x="11.2268" y="7.4168" extent="1-16" drill="0.6"/>
+<via x="18.2626" y="13.1572" extent="1-16" drill="0.6"/>
+<via x="15.4178" y="15.0114" extent="1-16" drill="0.6"/>
+<via x="18.5674" y="17.8308" extent="1-16" drill="0.5" diameter="0.254"/>
+<via x="15.5956" y="18.9484" extent="1-16" drill="0.5" diameter="0.254"/>
+<via x="11.7602" y="18.9484" extent="1-16" drill="0.5" diameter="0.254"/>
+<via x="12.8778" y="14.986" extent="1-16" drill="0.6"/>
+<via x="8.128" y="11.4046" extent="1-16" drill="0.6"/>
+<via x="5.0038" y="12.2174" extent="1-16" drill="0.6"/>
+<via x="6.223" y="19.1516" extent="1-16" drill="0.5" diameter="0.254"/>
 </signal>
 <signal name="ANALOG">
@@
 <wire x1="3.59588125" y1="13.4747" x2="3.59588125" y2="8.9497" width="0.4064" layer="1"/>
 </signal>
-<signal name="N$1">
-<via x="7.1374" y="7.5692" extent="1-16" drill="0.6"/>
-</signal>
-<signal name="N$2">
-<via x="5.3848" y="8.6614" extent="1-16" drill="0.6"/>
-</signal>
-<signal name="N$4">
-<via x="5.5372" y="5.8166" extent="1-16" drill="0.6"/>
-</signal>
-<signal name="N$5">
-<via x="15.4178" y="15.0114" extent="1-16" drill="0.6"/>
-</signal>
-<signal name="N$6">
-<via x="4.445" y="14.8844" extent="1-16" drill="0.6"/>
-</signal>
-<signal name="N$7">
-<via x="2.4384" y="14.2494" extent="1-16" drill="0.6"/>
-</signal>
-<signal name="N$8">
-<via x="9.6774" y="7.7216" extent="1-16" drill="0.6"/>
-</signal>
-<signal name="N$9">
-<via x="15.2908" y="4.0386" extent="1-16" drill="0.6"/>
-</signal>
-<signal name="N$10">
-<via x="5.3848" y="10.7696" extent="1-16" drill="0.6"/>
-</signal>
-<signal name="N$11">
-<via x="14.224" y="9.5758" extent="1-16" drill="0.6"/>
-</signal>
-<signal name="N$12">
-<via x="12.2174" y="11.3792" extent="1-16" drill="0.6"/>
-</signal>
-<signal name="N$13">
-<via x="8.128" y="11.4046" extent="1-16" drill="0.6"/>
-</signal>
-<signal name="N$14">
-<via x="8.4074" y="14.9606" extent="1-16" drill="0.6"/>
-</signal>
-<signal name="N$15">
-<via x="10.9728" y="5.0546" extent="1-16" drill="0.6"/>
-</signal>
-<signal name="N$16">
-<via x="15.5448" y="11.4046" extent="1-16" drill="0.6"/>
-</signal>
-<signal name="N$17">
-<via x="17.5006" y="13.208" extent="1-16" drill="0.6"/>
-</signal>
-<signal name="N$18">
-<via x="7.7978" y="9.525" extent="1-16" drill="0.6"/>
-</signal>
-<signal name="N$19">
-<via x="4.1148" y="3.7846" extent="1-16" drill="0.6"/>
-</signal>
-<signal name="N$20">
-<via x="12.8778" y="14.986" extent="1-16" drill="0.6"/>
-</signal>
-<signal name="N$21">
-<via x="5.0038" y="12.2174" extent="1-16" drill="0.6"/>
-</signal>
-<signal name="N$22">
-<via x="11.2268" y="7.4168" extent="1-16" drill="0.6"/>
-</signal>
-<signal name="N$23">
-<via x="13.843" y="4.5212" extent="1-16" drill="0.6"/>
-</signal>
-<signal name="N$24">
-<via x="2.5908" y="11.7348" extent="1-16" drill="0.6"/>
-</signal>
-<signal name="N$25">
-<via x="17.6022" y="10.4648" extent="1-16" drill="0.6"/>
-</signal>
-<signal name="N$26">
-<via x="3.2512" y="17.2212" extent="1-16" drill="0.6"/>
-</signal>
-<signal name="N$27">
-<via x="17.4244" y="16.4592" extent="1-16" drill="0.6"/>
-</signal>
-<signal name="N$28">
-<via x="8.5598" y="5.0038" extent="1-16" drill="0.5" diameter="0.254"/>
-</signal>
-<signal name="N$29">
-<via x="1.524" y="3.6068" extent="1-16" drill="0.5" diameter="0.254"/>
-</signal>
-<signal name="N$30">
-<via x="1.27" y="1.651" extent="1-16" drill="0.5" diameter="0.254"/>
-</signal>
-<signal name="N$31">
-<via x="2.4384" y="1.2192" extent="1-16" drill="0.5" diameter="0.254"/>
-</signal>
-<signal name="N$32">
-<via x="18.0848" y="2.1844" extent="1-16" drill="0.5" diameter="0.254"/>
-</signal>
-<signal name="N$33">
-<via x="14.7066" y="1.3462" extent="1-16" drill="0.5" diameter="0.254"/>
-</signal>
-<signal name="N$34">
-<via x="16.3576" y="1.4478" extent="1-16" drill="0.5" diameter="0.254"/>
-</signal>
-<signal name="N$35">
-<via x="18.9992" y="9.6012" extent="1-16" drill="0.5" diameter="0.254"/>
-</signal>
-<signal name="N$36">
-<via x="19.0246" y="12.7762" extent="1-16" drill="0.5" diameter="0.254"/>
-</signal>
-<signal name="N$37">
-<via x="19.1516" y="15.1638" extent="1-16" drill="0.5" diameter="0.254"/>
-</signal>
-<signal name="N$38">
-<via x="18.1864" y="14.6304" extent="1-16" drill="0.5" diameter="0.254"/>
-</signal>
-<signal name="N$39">
-<via x="18.5674" y="17.8308" extent="1-16" drill="0.5" diameter="0.254"/>
-</signal>
-<signal name="N$40">
-<via x="15.5956" y="18.9484" extent="1-16" drill="0.5" diameter="0.254"/>
-</signal>
-<signal name="N$41">
-<via x="11.7602" y="18.9484" extent="1-16" drill="0.5" diameter="0.254"/>
-</signal>
-<signal name="N$42">
-<via x="19.177" y="3.8608" extent="1-16" drill="0.5" diameter="0.254"/>
-</signal>
-<signal name="N$43">
-<via x="1.4986" y="18.3896" extent="1-16" drill="0.5" diameter="0.254"/>
-</signal>
-<signal name="N$44">
-<via x="6.223" y="19.1516" extent="1-16" drill="0.5" diameter="0.254"/>
-</signal>
 </signals>

Commit message: Updating/Cleaning-up documents
Other:
- board text added: "Analog"
- board text added: "Colten Nye,Steve Peirce,Golriz Sedaghat"
- board text added: "GND"
- board text added: "VCC"
- board text removed: "Colten Nye, Steve Peirce, Golriz Sedaghat"
Changed lines of the file:
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@@
 <setting verticaltext="up"/>
 </settings>
-<grid distance="0.001" unitdist="inch" unit="inch" style="lines" multiple="1" display="no" altdistance="0.025" altunitdist="inch" altunit="inch"/>
+<grid distance="0.01" unitdist="inch" unit="inch" style="lines" multiple="1" display="no" altdistance="0.025" altunitdist="inch" altunit="inch"/>
 <layers>
 <layer number="1" name="Top" color="4" fill="1" visible="yes" active="yes"/>
@@
 <wire x1="0" y1="20.292259375" x2="0" y2="0" width="0" layer="20"/>
 <text x="0.66801875" y="18.521678125" size="0.6096" layer="25">VOC Sensor Board </text>
-<text x="0.66548125" y="17.0053" size="0.6096" layer="25">Colten Nye, Steve Peirce, Golriz Sedaghat</text>
+<text x="0.66548125" y="17.0053" size="0.6096" layer="25">Colten Nye,Steve Peirce,Golriz Sedaghat</text>
+<text x="11.63828125" y="0.5715" size="0.6096" layer="25">GND</text>
+<text x="5.69468125" y="0.5969" size="0.6096" layer="25">VCC</text>
+<text x="8.13308125" y="0.5715" size="0.6096" layer="25">Analog</text>
 </plain>
 <attributes>
@@
 <polygon width="0.4064" layer="1">
 <vertex x="0" y="20.32"/>
-<vertex x="20.32" y="20.32"/>
-<vertex x="20.32" y="0"/>
+<vertex x="20.066" y="20.32"/>
+<vertex x="20.066" y="0"/>
 <vertex x="0" y="0"/>
-<vertex x="0" y="1.27"/>
 </polygon>
 <polygon width="0.4064" layer="16">
-<vertex x="0" y="20.32"/>
-<vertex x="20.32" y="20.32"/>
-<vertex x="20.32" y="0"/>
-<vertex x="0" y="0"/>
+<vertex x="0.0254" y="20.32"/>
+<vertex x="20.1168" y="20.3454"/>
+<vertex x="20.066" y="0"/>
+<vertex x="0.0254" y="0"/>
 </polygon>
 <via x="1.4986" y="18.3896" extent="1-16" drill="0.5" diameter="0.254"/>
